File: Tubes.brd (EAGLE design)
At the start: 100 x 80 mm, 26 parts, among them T0 MPSA42, T1 MPSA42, T2 MPSA42, T3 MPSA42, T4 MPSA42, T5 MPSA42, T6 MPSA42, T7 MPSA42, T8 MPSA42, T9 MPSA42

Commit message: Starting routing
Parts:
- moved HOURS_U 125.6 mm to (63.5, 69.8)
- moved R8 86.7 mm to (24.1, 21.6), turned to 0 degrees
- moved R9 80.7 mm to (24.1, 25.4), turned to 0 degrees
- moved R10 75.5 mm to (24.1, 29.2), turned to 0 degrees
- moved R11 71.5 mm to (24.1, 33.0), turned to 0 degrees
- moved R12 68.7 mm to (24.1, 36.8), turned to 0 degrees
- moved T6 65.9 mm to (41.9, 21.6)
- moved T7 62.0 mm to (35.6, 25.4)
- moved R1 54.0 mm to (91.4, 24.1)
- moved T8 50.3 mm to (41.9, 29.2)
- moved T9 49.5 mm to (35.6, 33.0)
- moved HOURS 43.0 mm to (11.4, 38.1), turned to 90 degrees
- moved T0 39.4 mm to (41.9, 36.8)
- moved POWER_SUPPLY 36.1 mm to (78.7, 17.8)
- moved T4 20.7 mm to (41.9, 52.1), turned to 270 degrees
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Connections:
- new net DIGIT_U0: HOURS.9, R12.1
- new net DIGIT_U1: HOURS.11, R3.1
- new net DIGIT_U2: HOURS.13, R4.1
- new net DIGIT_U3: HOURS.15, R5.1
- new net DIGIT_U4: HOURS.17, R6.1
- new net DIGIT_U5: HOURS.19, R7.1
- new net DIGIT_U6: HOURS.1, R8.1
- new net DIGIT_U7: HOURS.3, R9.1
- new net DIGIT_U8: HOURS.5, R10.1
- new net DIGIT_U9: HOURS.7, R11.1

Commit message: Keep routing
Parts:
- moved POWER_SUPPLY 75.5 mm to (24.1, 69.8), turned to 180 degrees
- moved R1 71.1 mm to (38.1, 71.1), turned to 270 degrees
- moved T5 66.5 mm to (83.8, 10.2)
- moved R7 65.1 mm to (86.4, 74.9)
- moved R6 61.4 mm to (82.5, 71.1)
- moved T4 59.7 mm to (88.9, 15.2)
- moved R5 59.0 mm to (80.0, 67.3)
- moved R4 56.6 mm to (77.5, 63.5)
- moved T3 55.8 mm to (83.8, 20.3)
- moved HOURS_U 55.1 mm to (71.1, 15.2), turned to 180 degrees
- moved R3 54.3 mm to (74.9, 59.7)
- moved HOURS_D 54.0 mm to (19.1, 19.1)
- moved R12 52.4 mm to (72.4, 57.1)
- moved T2 50.2 mm to (88.9, 26.7)
- moved R11 47.7 mm to (67.3, 53.3)
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Connections:
- net N$1: now also HOURS_U.0; no longer HOURS_D.0
- net N$13: now also HOURS_U.8; no longer HOURS_D.8
- net N$14: now also HOURS_U.7; no longer HOURS_D.7
- net N$15: now also HOURS_U.6; no longer HOURS_D.6
- net N$16: now also HOURS_U.5; no longer HOURS_D.5
- net N$17: now also HOURS_U.1; no longer HOURS_D.1
- net N$18: now also HOURS_U.4; no longer HOURS_D.4
- net N$19: now also HOURS_U.2; no longer HOURS_D.2
- net N$2: now also HOURS_U.9; no longer HOURS_D.9
- net N$21: now also HOURS_U.3; no longer HOURS_D.3
- net N$23: now also HOURS_U.A; no longer HOURS_D.A

Commit message: Complete schematics
Parts:
- added R13, R14, R15, R16, R17, R18, R19, R20, R21, R22: (no value), resistor:0207/10
- added T10, T11, T12, T13, T14, T15, T16, T17, T18, T19: MPSA42, PGT:TO92
- moved R2 80.7 mm to (30.5, 77.5), turned to 180 degrees
- moved R8 29.2 mm to (64.8, 47.0), turned to 0 degrees
- moved R7 22.2 mm to (64.8, 69.8)
- moved R9 19.0 mm to (64.8, 49.5), turned to 0 degrees
- moved POWER_SUPPLY 18.9 mm to (41.9, 76.2)
- moved R6 18.2 mm to (64.8, 67.3)
- moved R1 17.7 mm to (54.6, 77.5), turned to 0 degrees
- moved R5 15.5 mm to (64.8, 64.8)
- moved R4 12.8 mm to (64.8, 62.2)
- moved T7 12.8 mm to (47.0, 17.8)
- moved T8 12.8 mm to (47.0, 25.4)
- moved T6 12.7 mm to (47.0, 10.2)
- moved HOURS_U 11.4 mm to (59.7, 15.2)
- moved T1 11.4 mm to (69.8, 31.8)
- moved T2 11.4 mm to (77.5, 26.7)
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Connections:
- new net DIGIT_D0: HOURS.10, R22.1
- new net DIGIT_D1: HOURS.12, R13.1
- new net DIGIT_D2: HOURS.14, R14.1
- new net DIGIT_D3: HOURS.16, R15.1
- new net DIGIT_D4: HOURS.18, R16.1
- new net DIGIT_D5: HOURS.20, R17.1
- new net DIGIT_D6: HOURS.2, R18.1
- new net DIGIT_D7: HOURS.4, R19.1
- new net DIGIT_D8: HOURS.6, R20.1
- new net DIGIT_D9: HOURS.8, R21.1
- new net N$20: HOURS_D.0, T10.3
- new net N$22: HOURS_D.9, T19.3
- new net N$24: HOURS_D.8, T18.3
- new net N$25: HOURS_D.7, T17.3
- new net N$26: HOURS_D.6, T16.3
- new net N$27: HOURS_D.5, T15.3
- new net N$28: HOURS_D.2, T12.3
- new net N$29: HOURS_D.A, R2.2
- new net N$30: HOURS_D.3, T13.3
- new net N$31: HOURS_D.4, T14.3
- new net N$32: HOURS_D.1, T11.3
- new net N$33: R17.2, T15.2
- new net N$34: R18.2, T16.2
- new net N$35: R19.2, T17.2
- new net N$36: R22.2, T10.2
- new net N$37: R13.2, T11.2
- new net N$38: R15.2, T13.2
- new net N$39: R14.2, T12.2
- new net N$40: R16.2, T14.2
- new net N$41: R20.2, T18.2
- new net N$42: R21.2, T19.2
- net GND: now also T10.1, T11.1, T12.1, T13.1, T14.1, T15.1, T16.1, T17.1, T18.1, T19.1
- net VCC: now also R2.1
