File: Tubes.sch (EAGLE design)
At the start: 26 parts, among them T0 MPSA42, T1 MPSA42, T2 MPSA42, T3 MPSA42, T4 MPSA42, T5 MPSA42, T6 MPSA42, T7 MPSA42, T8 MPSA42, T9 MPSA42

Commit message: Create tube board
Connections:
- new net N$1: HOURS_D.0, T0.C
- new net N$13: HOURS_D.8, T8.C
- new net N$14: HOURS_D.7, T7.C
- new net N$15: HOURS_D.6, T6.C
- new net N$16: HOURS_D.5, T5.C
- new net N$18: HOURS_D.4, T4.C
- new net N$19: HOURS_D.2, T2.C
- new net N$2: HOURS_D.9, T9.C
- new net N$20: HOURS_D.1, T1.C
- new net N$21: HOURS_D.3, T3.C
- new net N$23: HOURS_D.A, R1.2
- net VCC: now also R1.1
Other:
- moved on the sheet: R1, R2
Changed lines of the file:
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@@
 <instance part="HOURS_U" gate="G$1" x="27.94" y="91.44" rot="R270"/>
 <instance part="HOURS" gate="A" x="81.28" y="91.44" rot="R270"/>
-<instance part="R2" gate="G$1" x="25.4" y="73.66" rot="R90"/>
-<instance part="R1" gate="G$1" x="121.92" y="106.68" rot="R90"/>
+<instance part="R2" gate="G$1" x="2.54" y="91.44" rot="R90"/>
+<instance part="R1" gate="G$1" x="137.16" y="104.14" rot="R180"/>
 <instance part="HOURS_D" gate="G$1" x="129.54" y="88.9" rot="R90"/>
 <instance part="POWER_SUPPLY" gate="G$1" x="10.16" y="162.56"/>
 <instance part="SUPPLY1" gate="GND" x="33.02" y="152.4"/>
 <instance part="P+1" gate="VCC" x="33.02" y="172.72"/>
-<instance part="P+2" gate="VCC" x="137.16" y="106.68"/>
-<instance part="P+3" gate="VCC" x="25.4" y="63.5" rot="R180"/>
+<instance part="P+2" gate="VCC" x="144.78" y="109.22"/>
+<instance part="P+3" gate="VCC" x="-7.62" y="91.44" rot="R180"/>
 <instance part="T1" gate="G$1" x="15.24" y="30.48"/>
 <instance part="T2" gate="G$1" x="30.48" y="30.48"/>
@@
 <wire x1="33.02" y1="165.1" x2="33.02" y2="170.18" width="0.1524" layer="91"/>
 </segment>
+<segment>
+<pinref part="R1" gate="G$1" pin="1"/>
+<pinref part="P+2" gate="VCC" pin="VCC"/>
+<wire x1="142.24" y1="104.14" x2="144.78" y2="104.14" width="0.1524" layer="91"/>
+<wire x1="144.78" y1="104.14" x2="144.78" y2="106.68" width="0.1524" layer="91"/>
+</segment>
 </net>
 <net name="N$3" class="0">
@@
 </segment>
 </net>
+<net name="N$1" class="0">
+<segment>
+<pinref part="HOURS_D" gate="G$1" pin="0"/>
+<wire x1="142.24" y1="81.28" x2="142.24" y2="55.88" width="0.1524" layer="91"/>
+<wire x1="142.24" y1="55.88" x2="154.94" y2="55.88" width="0.1524" layer="91"/>
+<pinref part="T0" gate="G$1" pin="C"/>
+<wire x1="154.94" y1="55.88" x2="154.94" y2="35.56" width="0.1524" layer="91"/>
+</segment>
+</net>
+<net name="N$2" class="0">
+<segment>
+<pinref part="HOURS_D" gate="G$1" pin="9"/>
+<wire x1="139.7" y1="81.28" x2="139.7" y2="35.56" width="0.1524" layer="91"/>
+<pinref part="T9" gate="G$1" pin="C"/>
+</segment>
+</net>
+<net name="N$13" class="0">
+<segment>
+<pinref part="HOURS_D" gate="G$1" pin="8"/>
+<wire x1="137.16" y1="81.28" x2="137.16" y2="55.88" width="0.1524" layer="91"/>
+<wire x1="137.16" y1="55.88" x2="124.46" y2="55.88" width="0.1524" layer="91"/>
+<pinref part="T8" gate="G$1" pin="C"/>
+<wire x1="124.46" y1="55.88" x2="124.46" y2="35.56" width="0.1524" layer="91"/>
+</segment>
+</net>
+<net name="N$14" class="0">
+<segment>
+<pinref part="HOURS_D" gate="G$1" pin="7"/>
+<wire x1="134.62" y1="81.28" x2="134.62" y2="58.42" width="0.1524" layer="91"/>
+<pinref part="T7" gate="G$1" pin="C"/>
+<wire x1="134.62" y1="58.42" x2="109.22" y2="58.42" width="0.1524" layer="91"/>
+<wire x1="109.22" y1="58.42" x2="109.22" y2="35.56" width="0.1524" layer="91"/>
+</segment>
+</net>
+<net name="N$15" class="0">
+<segment>
+<pinref part="HOURS_D" gate="G$1" pin="6"/>
+<wire x1="132.08" y1="81.28" x2="132.08" y2="60.96" width="0.1524" layer="91"/>
+<pinref part="T6" gate="G$1" pin="C"/>
+<wire x1="132.08" y1="60.96" x2="93.98" y2="60.96" width="0.1524" layer="91"/>
+<wire x1="93.98" y1="60.96" x2="93.98" y2="35.56" width="0.1524" layer="91"/>
+</segment>
+</net>
+<net name="N$16" class="0">
+<segment>
+<pinref part="HOURS_D" gate="G$1" pin="5"/>
+<wire x1="129.54" y1="81.28" x2="129.54" y2="63.5" width="0.1524" layer="91"/>
+<pinref part="T5" gate="G$1" pin="C"/>
+<wire x1="129.54" y1="63.5" x2="78.74" y2="63.5" width="0.1524" layer="91"/>
+<wire x1="78.74" y1="63.5" x2="78.74" y2="35.56" width="0.1524" layer="91"/>
+</segment>
+</net>
+<net name="N$19" class="0">
+<segment>
+<pinref part="HOURS_D" gate="G$1" pin="2"/>
+<wire x1="121.92" y1="81.28" x2="121.92" y2="71.12" width="0.1524" layer="91"/>
+<pinref part="T2" gate="G$1" pin="C"/>
+<wire x1="121.92" y1="71.12" x2="33.02" y2="71.12" width="0.1524" layer="91"/>
+<wire x1="33.02" y1="71.12" x2="33.02" y2="35.56" width="0.1524" layer="91"/>
+</segment>
+</net>
+<net name="N$20" class="0">
+<segment>
+<pinref part="HOURS_D" gate="G$1" pin="1"/>
+<wire x1="119.38" y1="81.28" x2="119.38" y2="73.66" width="0.1524" layer="91"/>
+<pinref part="T1" gate="G$1" pin="C"/>
+<wire x1="119.38" y1="73.66" x2="17.78" y2="73.66" width="0.1524" layer="91"/>
+<wire x1="17.78" y1="73.66" x2="17.78" y2="35.56" width="0.1524" layer="91"/>
+</segment>
+</net>
+<net name="N$23" class="0">
+<segment>
+<pinref part="R1" gate="G$1" pin="2"/>
+<pinref part="HOURS_D" gate="G$1" pin="A"/>
+<wire x1="132.08" y1="104.14" x2="132.08" y2="99.06" width="0.1524" layer="91"/>
+</segment>
+</net>
+<net name="N$21" class="0">
+<segment>
+<pinref part="HOURS_D" gate="G$1" pin="3"/>
+<wire x1="124.46" y1="81.28" x2="124.46" y2="68.58" width="0.1524" layer="91"/>
+<pinref part="T3" gate="G$1" pin="C"/>
+<wire x1="124.46" y1="68.58" x2="48.26" y2="68.58" width="0.1524" layer="91"/>
+<wire x1="48.26" y1="68.58" x2="48.26" y2="35.56" width="0.1524" layer="91"/>
+</segment>
+</net>
+<net name="N$18" class="0">
+<segment>
+<pinref part="HOURS_D" gate="G$1" pin="4"/>
+<wire x1="127" y1="81.28" x2="127" y2="66.04" width="0.1524" layer="91"/>
+<pinref part="T4" gate="G$1" pin="C"/>
+<wire x1="127" y1="66.04" x2="63.5" y2="66.04" width="0.1524" layer="91"/>
+<wire x1="63.5" y1="66.04" x2="63.5" y2="35.56" width="0.1524" layer="91"/>
+</segment>
+</net>

Commit message: Starting routing
Connections:
- new net DIGIT_U0: HOURS.9, R12.1
- new net DIGIT_U1: HOURS.11, R3.1
- new net DIGIT_U2: HOURS.13, R4.1
- new net DIGIT_U3: HOURS.15, R5.1
- new net DIGIT_U4: HOURS.17, R6.1
- new net DIGIT_U5: HOURS.19, R7.1
- new net DIGIT_U6: HOURS.1, R8.1
- new net DIGIT_U7: HOURS.3, R9.1
- new net DIGIT_U8: HOURS.5, R10.1
- new net DIGIT_U9: HOURS.7, R11.1
Other:
- moved on the sheet: HOURS
Changed lines of the file:
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@@
 <instance part="FRAME1" gate="G$2" x="162.56" y="0"/>
 <instance part="HOURS_U" gate="G$1" x="27.94" y="91.44" rot="R270"/>
-<instance part="HOURS" gate="A" x="81.28" y="91.44" rot="R270"/>
+<instance part="HOURS" gate="A" x="198.12" y="147.32" rot="R180"/>
 <instance part="R2" gate="G$1" x="2.54" y="91.44" rot="R90"/>
 <instance part="R1" gate="G$1" x="137.16" y="104.14" rot="R180"/>
@@
 </segment>
 </net>
-<net name="N$20" class="0">
+<net name="N$23" class="0">
+<segment>
+<pinref part="R1" gate="G$1" pin="2"/>
+<pinref part="HOURS_D" gate="G$1" pin="A"/>
+<wire x1="132.08" y1="104.14" x2="132.08" y2="99.06" width="0.1524" layer="91"/>
+</segment>
+</net>
+<net name="N$21" class="0">
+<segment>
+<pinref part="HOURS_D" gate="G$1" pin="3"/>
+<wire x1="124.46" y1="81.28" x2="124.46" y2="68.58" width="0.1524" layer="91"/>
+<pinref part="T3" gate="G$1" pin="C"/>
+<wire x1="124.46" y1="68.58" x2="48.26" y2="68.58" width="0.1524" layer="91"/>
+<wire x1="48.26" y1="68.58" x2="48.26" y2="35.56" width="0.1524" layer="91"/>
+</segment>
+</net>
+<net name="N$18" class="0">
+<segment>
+<pinref part="HOURS_D" gate="G$1" pin="4"/>
+<wire x1="127" y1="81.28" x2="127" y2="66.04" width="0.1524" layer="91"/>
+<pinref part="T4" gate="G$1" pin="C"/>
+<wire x1="127" y1="66.04" x2="63.5" y2="66.04" width="0.1524" layer="91"/>
+<wire x1="63.5" y1="66.04" x2="63.5" y2="35.56" width="0.1524" layer="91"/>
+</segment>
+</net>
+<net name="DIGIT_U1" class="0">
+<segment>
+<pinref part="R3" gate="G$1" pin="1"/>
+<wire x1="10.16" y1="50.8" x2="10.16" y2="53.34" width="0.1524" layer="91"/>
+<label x="10.16" y="53.34" size="1.778" layer="95"/>
+</segment>
+<segment>
+<pinref part="HOURS" gate="A" pin="11"/>
+<wire x1="175.26" y1="147.32" x2="190.5" y2="147.32" width="0.1524" layer="91"/>
+<label x="175.26" y="147.32" size="1.778" layer="95"/>
+</segment>
+</net>
+<net name="DIGIT_U2" class="0">
+<segment>
+<pinref part="R4" gate="G$1" pin="1"/>
+<wire x1="25.4" y1="50.8" x2="25.4" y2="53.34" width="0.1524" layer="91"/>
+<label x="25.4" y="53.34" size="1.778" layer="95"/>
+</segment>
+<segment>
+<pinref part="HOURS" gate="A" pin="13"/>
+<wire x1="175.26" y1="144.78" x2="190.5" y2="144.78" width="0.1524" layer="91"/>
+<label x="175.26" y="144.78" size="1.778" layer="95"/>
+</segment>
+</net>
+<net name="DIGIT_U3" class="0">
+<segment>
+<pinref part="R5" gate="G$1" pin="1"/>
+<wire x1="40.64" y1="50.8" x2="40.64" y2="53.34" width="0.1524" layer="91"/>
+<label x="40.64" y="53.34" size="1.778" layer="95"/>
+</segment>
+<segment>
+<pinref part="HOURS" gate="A" pin="15"/>
+<wire x1="175.26" y1="142.24" x2="190.5" y2="142.24" width="0.1524" layer="91"/>
+<label x="175.26" y="142.24" size="1.778" layer="95"/>
+</segment>
+</net>
+<net name="DIGIT_U4" class="0">
+<segment>
+<pinref part="R6" gate="G$1" pin="1"/>
+<wire x1="55.88" y1="50.8" x2="55.88" y2="53.34" width="0.1524" layer="91"/>
+<label x="55.88" y="53.34" size="1.778" layer="95"/>
+</segment>
+<segment>
+<pinref part="HOURS" gate="A" pin="17"/>
+<wire x1="175.26" y1="139.7" x2="190.5" y2="139.7" width="0.1524" layer="91"/>
+<label x="175.26" y="139.7" size="1.778" layer="95"/>
+</segment>
+</net>
+<net name="DIGIT_U5" class="0">
+<segment>
+<pinref part="R7" gate="G$1" pin="1"/>
+<wire x1="71.12" y1="50.8" x2="71.12" y2="53.34" width="0.1524" layer="91"/>
+<label x="71.12" y="53.34" size="1.778" layer="95"/>
+</segment>
+<segment>
+<pinref part="HOURS" gate="A" pin="19"/>
+<wire x1="190.5" y1="137.16" x2="175.26" y2="137.16" width="0.1524" layer="91"/>
+<label x="175.26" y="137.16" size="1.778" layer="95"/>
+</segment>
+</net>
+<net name="DIGIT_U6" class="0">
+<segment>
+<pinref part="R8" gate="G$1" pin="1"/>
+<wire x1="86.36" y1="50.8" x2="86.36" y2="53.34" width="0.1524" layer="91"/>
+<label x="86.36" y="53.34" size="1.778" layer="95"/>
+</segment>
+<segment>
+<pinref part="HOURS" gate="A" pin="1"/>
+<wire x1="190.5" y1="160.02" x2="175.26" y2="160.02" width="0.1524" layer="91"/>
+<label x="175.26" y="160.02" size="1.778" layer="95"/>
+</segment>
+</net>
+<net name="DIGIT_U8" class="0">
+<segment>
+<pinref part="R10" gate="G$1" pin="1"/>
+<wire x1="116.84" y1="50.8" x2="116.84" y2="53.34" width="0.1524" layer="91"/>
+<label x="116.84" y="53.34" size="1.778" layer="95"/>
+</segment>
+<segment>
+<pinref part="HOURS" gate="A" pin="5"/>
+<wire x1="190.5" y1="154.94" x2="175.26" y2="154.94" width="0.1524" layer="91"/>
+<label x="175.26" y="154.94" size="1.778" layer="95"/>
+</segment>
+</net>
+<net name="DIGIT_U9" class="0">
+<segment>
+<pinref part="R11" gate="G$1" pin="1"/>
+<wire x1="132.08" y1="50.8" x2="132.08" y2="53.34" width="0.1524" layer="91"/>
+<label x="132.08" y="53.34" size="1.778" layer="95"/>
+</segment>
+<segment>
+<pinref part="HOURS" gate="A" pin="7"/>
+<wire x1="190.5" y1="152.4" x2="175.26" y2="152.4" width="0.1524" layer="91"/>
+<label x="175.26" y="152.4" size="1.778" layer="95"/>
+</segment>
+</net>
+<net name="DIGIT_U0" class="0">
+<segment>
+<pinref part="R12" gate="G$1" pin="1"/>
+<wire x1="147.32" y1="50.8" x2="147.32" y2="53.34" width="0.1524" layer="91"/>
+<label x="147.32" y="53.34" size="1.778" layer="95"/>
+</segment>
+<segment>
+<pinref part="HOURS" gate="A" pin="9"/>
+<wire x1="190.5" y1="149.86" x2="175.26" y2="149.86" width="0.1524" layer="91"/>
+<label x="175.26" y="149.86" size="1.778" layer="95"/>
+</segment>
+</net>
+<net name="DIGIT_U7" class="0">
+<segment>
+<pinref part="R9" gate="G$1" pin="1"/>
+<wire x1="101.6" y1="50.8" x2="101.6" y2="53.34" width="0.1524" layer="91"/>
+<label x="101.6" y="53.34" size="1.778" layer="95"/>
+</segment>
+<segment>
+<pinref part="HOURS" gate="A" pin="3"/>
+<wire x1="190.5" y1="157.48" x2="175.26" y2="157.48" width="0.1524" layer="91"/>
+<label x="175.26" y="157.48" size="1.778" layer="95"/>
+</segment>
+</net>
+<net name="N$17" class="0">
 <segment>
 <pinref part="HOURS_D" gate="G$1" pin="1"/>
@@
 </segment>
 </net>
-<net name="N$23" class="0">
-<segment>
-<pinref part="R1" gate="G$1" pin="2"/>
-<pinref part="HOURS_D" gate="G$1" pin="A"/>
-<wire x1="132.08" y1="104.14" x2="132.08" y2="99.06" width="0.1524" layer="91"/>
-</segment>
-</net>
-<net name="N$21" class="0">
-<segment>
-<pinref part="HOURS_D" gate="G$1" pin="3"/>
-<wire x1="124.46" y1="81.28" x2="124.46" y2="68.58" width="0.1524" layer="91"/>
-<pinref part="T3" gate="G$1" pin="C"/>
-<wire x1="124.46" y1="68.58" x2="48.26" y2="68.58" width="0.1524" layer="91"/>
-<wire x1="48.26" y1="68.58" x2="48.26" y2="35.56" width="0.1524" layer="91"/>
-</segment>
-</net>
-<net name="N$18" class="0">
-<segment>
-<pinref part="HOURS_D" gate="G$1" pin="4"/>
-<wire x1="127" y1="81.28" x2="127" y2="66.04" width="0.1524" layer="91"/>
-<pinref part="T4" gate="G$1" pin="C"/>
-<wire x1="127" y1="66.04" x2="63.5" y2="66.04" width="0.1524" layer="91"/>
-<wire x1="63.5" y1="66.04" x2="63.5" y2="35.56" width="0.1524" layer="91"/>
-</segment>
-</net>

Commit message: Keep routing
Connections:
- net N$1: now also HOURS_U.0; no longer HOURS_D.0
- net N$13: now also HOURS_U.8; no longer HOURS_D.8
- net N$14: now also HOURS_U.7; no longer HOURS_D.7
- net N$15: now also HOURS_U.6; no longer HOURS_D.6
- net N$16: now also HOURS_U.5; no longer HOURS_D.5
- net N$17: now also HOURS_U.1; no longer HOURS_D.1
- net N$18: now also HOURS_U.4; no longer HOURS_D.4
- net N$19: now also HOURS_U.2; no longer HOURS_D.2
- net N$2: now also HOURS_U.9; no longer HOURS_D.9
- net N$21: now also HOURS_U.3; no longer HOURS_D.3
- net N$23: now also HOURS_U.A; no longer HOURS_D.A
Other:
- moved on the sheet: HOURS_D, HOURS_U

Commit message: Complete schematics
Parts:
- added R13, R14, R15, R16, R17, R18, R19, R20, R21, R22: (no value), resistor:R-EU_0207/10
- added T10, T11, T12, T13, T14, T15, T16, T17, T18, T19: MPSA42, PGT:MPSA42
Connections:
- new net DIGIT_D0: HOURS.10, R22.1
- new net DIGIT_D1: HOURS.12, R13.1
- new net DIGIT_D2: HOURS.14, R14.1
- new net DIGIT_D3: HOURS.16, R15.1
- new net DIGIT_D4: HOURS.18, R16.1
- new net DIGIT_D5: HOURS.20, R17.1
- new net DIGIT_D6: HOURS.2, R18.1
- new net DIGIT_D7: HOURS.4, R19.1
- new net DIGIT_D8: HOURS.6, R20.1
- new net DIGIT_D9: HOURS.8, R21.1
- new net N$20: HOURS_D.0, T10.C
- new net N$22: HOURS_D.9, T19.C
- new net N$24: HOURS_D.8, T18.C
- new net N$25: HOURS_D.7, T17.C
- new net N$26: HOURS_D.6, T16.C
- new net N$27: HOURS_D.5, T15.C
- new net N$28: HOURS_D.2, T12.C
- new net N$29: HOURS_D.A, R2.2
- new net N$30: HOURS_D.3, T13.C
- new net N$31: HOURS_D.4, T14.C
- new net N$32: HOURS_D.1, T11.C
- new net N$33: R17.2, T15.B
- new net N$34: R18.2, T16.B
- new net N$35: R19.2, T17.B
- new net N$36: R22.2, T10.B
- new net N$37: R13.2, T11.B
- new net N$38: R15.2, T13.B
- new net N$39: R14.2, T12.B
- new net N$40: R16.2, T14.B
- new net N$41: R20.2, T18.B
- new net N$42: R21.2, T19.B
- net GND: now also T10.E, T11.E, T12.E, T13.E, T14.E, T15.E, T16.E, T17.E, T18.E, T19.E
- net VCC: now also R2.1
Other:
- moved on the sheet: HOURS, HOURS_D, HOURS_U, POWER_SUPPLY, R1, R10, R11, R12, R2, R3, R4, R5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
