File: Nixie Clock.brd (EAGLE design)
At the start: 100 x 80 mm, 46 parts, among them T0 MPSA42, T1 MPSA42, T10 MPSA42, T11 MPSA42, T12 MPSA42, T13 MPSA42, T14 MPSA42, T15 MPSA42, T16 MPSA42, T17 MPSA42, T18 MPSA42, T19 MPSA42, T2 MPSA42, T3 MPSA42, T4 MPSA42, T5 MPSA42, T6 MPSA42, T7 MPSA42, T8 MPSA42, T9 MPSA42

Commit message: Create 'Nixie Clock' and delete previous attempts with tubes
Parts:
- removed HOURS: (no value), con-harting:CON20
- removed HOURS_D, HOURS_U: IN-14, russian-nixies:IN-14
- removed POWER_SUPPLY: CON_2_SIL, PGT:SIL_2_0.2INCH
- added CON_LOGIC_POWER, CON_TUBE_POWER: CON_2_SIL, PGT:SIL_2_0.2INCH
- added HOURS_TENS, HOURS_UNITS, MINUTES_TENS, MINUTES_UNITS, SECONDS_TENS, SECONDS_UNITS: IN-14, russian-nixies:IN-14
- added R23, R24, R25, R26, R27, R28, R29, R30, R31, R32, R33, R34, R35, R36, R39, R40, R41, R42, R43, R44, R45, R46, R47, R48, R49, R50, R54: 33.3k, resistor:0207/10
- added R37, R38: (no value), resistor:0207/10
- added T20, T21, T22, T23, T24, T25, T26, T27, T28, T29, T30, T31, T32, T33, T34, T35, T36, T37, T38, T39, T40, T41, T42, T43, T44: MPSA42, PGT:TO92
- R10, R11, R12, R13, R14, R15, R16, R17, R18, R21, R22, R3, R4, R5, R6, R7, R8, R9: value (none) -> 33.3k
- moved R22 311.2 mm to (31.8, -259.1), turned to 0 degrees
- moved R21 309.1 mm to (19.1, -259.1), turned to 0 degrees
- moved R20 307.5 mm to (6.35, -259.1), turned to 0 degrees
- moved R19 298.8 mm to (49.5, -254.0), turned to 0 degrees
- moved R17 270.8 mm to (6.35, -204.5), turned to 0 degrees
- moved T19 264.8 mm to (31.8, -238.8), turned to 0 degrees
- moved R16 263.2 mm to (6.35, -199.4), turned to 0 degrees
- moved T18 257.8 mm to (17.8, -238.8), turned to 0 degrees
- moved R15 255.7 mm to (6.35, -194.3), turned to 0 degrees
- moved R18 253.2 mm to (6.35, -209.6), turned to 0 degrees
- moved T17 251.7 mm to (3.81, -238.8), turned to 0 degrees
- moved R14 248.1 mm to (6.35, -189.2), turned to 0 degrees
- moved R13 240.5 mm to (6.35, -184.2), turned to 0 degrees
- moved R12 236.9 mm to (6.35, -179.1)
- moved R11 229.5 mm to (6.35, -174.0)
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Connections:
- removed net DIGIT_D0: HOURS.10, R22.1
- removed net DIGIT_D1: HOURS.12, R13.1
- removed net DIGIT_D2: HOURS.14, R14.1
- removed net DIGIT_D3: HOURS.16, R15.1
- removed net DIGIT_D4: HOURS.18, R16.1
- removed net DIGIT_D5: HOURS.20, R17.1
- removed net DIGIT_D6: HOURS.2, R18.1
- removed net DIGIT_D7: HOURS.4, R19.1
- removed net DIGIT_D8: HOURS.6, R20.1
- removed net DIGIT_D9: HOURS.8, R21.1
- removed net DIGIT_U0: HOURS.9, R12.1
- removed net DIGIT_U1: HOURS.11, R3.1
- removed net DIGIT_U2: HOURS.13, R4.1
- removed net DIGIT_U3: HOURS.15, R5.1
- removed net DIGIT_U4: HOURS.17, R6.1
- removed net DIGIT_U5: HOURS.19, R7.1
- removed net DIGIT_U6: HOURS.1, R8.1
- removed net DIGIT_U7: HOURS.3, R9.1
- removed net DIGIT_U8: HOURS.5, R10.1
- removed net DIGIT_U9: HOURS.7, R11.1
- removed net N$1 (its old number): HOURS_U.0, T0.3
- removed net N$13 (its old number): HOURS_U.8, T8.3
- removed net N$14 (its old number): HOURS_U.7, T7.3
- removed net N$16 (its old number): HOURS_U.5, T5.3
- removed net N$17 (its old number): HOURS_U.1, T1.3
- removed net N$18 (its old number): HOURS_U.4, T4.3
- removed net N$2 (its old number): HOURS_U.9, T9.3
- new net N$33: SECONDS_UNITS.9, T9.3
- new net N$37: R26.2, T21.2
- new net N$38: R27.2, T22.2
- new net N$39: R28.2, T23.2
- new net N$40: R29.2, T24.2
- new net N$43: MINUTES_TENS.A, R20.1
- new net N$44: R31.2, T27.2
- new net N$45: R32.2, T28.2
- new net N$46: R33.2, T29.2
- new net N$47: R34.2, T30.2
- new net N$48: R35.2, T31.2
- new net N$49: R36.2, T26.2
- new net N$50: R21.2, T16.2
- new net N$51: R22.2, T17.2
- new net N$52: R23.2, T18.2
- new net N$53: MINUTES_TENS.1, T27.3
- new net N$54: MINUTES_TENS.2, T28.3
- new net N$55: MINUTES_TENS.3, T29.3
- new net N$56: MINUTES_TENS.4, T30.3
- new net N$57: MINUTES_TENS.5, T31.3
- new net N$58: MINUTES_TENS.0, T26.3
- new net N$59: MINUTES_UNITS.1, T16.3
- new net N$60: MINUTES_UNITS.2, T17.3
- new net N$61: MINUTES_UNITS.3, T18.3
- new net N$62: MINUTES_UNITS.4, T19.3
- new net N$63: MINUTES_UNITS.5, T20.3
- new net N$64: MINUTES_UNITS.6, T21.3
- new net N$65: MINUTES_UNITS.0, T25.3
- new net N$66: MINUTES_UNITS.9, T24.3
- new net N$67: MINUTES_UNITS.8, T23.3
- new net N$68: R43.2, T36.2
- new net N$69: R44.2, T37.2
- new net N$70: R45.2, T38.2
- new net N$71: R46.2, T39.2
- new net N$72: R47.2, T40.2
- new net N$73: R48.2, T41.2
- new net N$74: HOURS_UNITS.A, R37.1
- new net N$75: HOURS_TENS.A, R38.1
- new net N$76: R49.2, T43.2
- new net N$77: R50.2, T44.2
- new net N$78: HOURS_TENS.0, T42.3
- new net N$8: R1.1, SECONDS_UNITS.A
- new net N$81: R54.2, T42.2
- new net N$82: R39.2, T32.2
- new net N$83: R40.2, T33.2
- new net N$84: R41.2, T34.2
- new net N$85: HOURS_TENS.1, T43.3
- new net N$86: HOURS_TENS.2, T44.3
- new net N$9: R2.1, SECONDS_TENS.A
- new net N$91: HOURS_UNITS.1, T32.3
- new net N$92: HOURS_UNITS.2, T33.3
- new net N$93: HOURS_UNITS.3, T34.3
- new net N$94: HOURS_UNITS.4, T35.3
- new net N$95: HOURS_UNITS.5, T36.3
- new net N$96: HOURS_UNITS.6, T37.3
- new net N$97: HOURS_UNITS.0, T41.3
- new net N$98: HOURS_UNITS.9, T40.3
- new net N$99: HOURS_UNITS.8, T39.3
- new net VHIGH: CON_TUBE_POWER.P$1, R1.2, R19.2, R2.2, R20.2, R37.2, R38.2
- net GND: now also CON_LOGIC_POWER.P$2, CON_TUBE_POWER.P$2, HOURS_UNITS.7, MINUTES_UNITS.7, SECONDS_UNITS.7, T20.1, T21.1, T22.1, T23.1, T24.1, T25.1, T26.1, T27.1, T28.1, T29.1, T30.1, T31.1, T32.1, T33.1, T34.1, T35.1, T36.1, T37.1, T38.1, T39.1, T40.1, T41.1, T42.1, T43.1, T44.1; no longer POWER_SUPPLY.P$2
- net N$15: now also R18.2, T10.2; no longer HOURS_U.6, T6.3
- net N$19: now also SECONDS_TENS.1, T11.3; no longer HOURS_U.2, T2.3
- net N$20: now also SECONDS_TENS.2, T12.3; no longer HOURS_D.0, T10.3
- net N$21: now also SECONDS_TENS.3, T13.3; no longer HOURS_U.3, T3.3
- net N$22: now also SECONDS_TENS.4, T14.3; no longer HOURS_D.9, T19.3
- net N$23: now also SECONDS_TENS.5, T15.3; no longer HOURS_U.A, R1.2
- net N$24: now also SECONDS_TENS.0, T10.3; no longer HOURS_D.8, T18.3
- net N$25: now also R42.2, T35.2; no longer HOURS_D.7, T17.3
- net N$26: now also SECONDS_UNITS.1, T1.3; no longer HOURS_D.6, T16.3
- net N$27: now also SECONDS_UNITS.2, T2.3; no longer HOURS_D.5, T15.3
- net N$28: now also SECONDS_UNITS.3, T3.3; no longer HOURS_D.2, T12.3
- net N$29: now also SECONDS_UNITS.4, T4.3; no longer HOURS_D.A, R2.2
- net N$30: now also SECONDS_UNITS.5, T5.3; no longer HOURS_D.3, T13.3
- net N$31: now also SECONDS_UNITS.6, T6.3; no longer HOURS_D.4, T14.3
- net N$32: now also SECONDS_UNITS.0, T0.3; no longer HOURS_D.1, T11.3
- net N$34: now also SECONDS_UNITS.8, T8.3; no longer R18.2, T16.2
- net N$35: now also R24.2, T19.2; no longer R19.2, T17.2
- net N$36: now also R25.2, T20.2; no longer R22.2, T10.2
- net N$41: now also R30.2, T25.2; no longer R20.2, T18.2
- net N$42: now also MINUTES_UNITS.A, R19.1; no longer R21.2, T19.2
- net VCC: now also CON_LOGIC_POWER.P$1; no longer POWER_SUPPLY.P$1, R1.1, R2.1
Other:
- board size 100 x 80 mm -> 182.6 x 80 mm

Commit message: Uncompleted schematics for the Nixie Clock and simulation for AND with diodes
Parts:
- removed CON_TUBE_POWER: CON_2_SIL, PGT:SIL_2_0.2INCH
- added C1, C2, C3, C4, C5, C6: 100n, resistor:C050-030X075
- added CON_HIGH_VOLTAGE, CON_TIME_REF: CON_2_SIL, PGT:SIL_2_0.2INCH
- added D1, D10, D11, D2, D3, D4, D5, D6, D7, D8, D9: 1N4148DO35-7, diode:DO35-7
- added IC1_SECONDS_UNITS, IC2_SECONDS_TENS, IC3_MINUTES_UNITS, IC4_MINUTES_TENS, IC5_HOURS_UNITS, IC6_HOURS_TENS: 4017N, 40xx:DIL16
- added R51, R52, R53, R55, R56, R57: 22k, resistor:0207/10
- added R58: 5k, resistor:0207/10
- added S1: SWITCH-MOMENTARY-2PTH, SparkFun-Electromechanical:TACTILE-PTH
- moved R19 303.2 mm to (86.4, 47.0)
- moved R2 185.8 mm to (86.4, 39.4)
- moved R1 184.6 mm to (86.4, 43.2)
- moved HOURS_TENS 36.3 mm to (83.8, 26.7)
- moved CON_LOGIC_POWER 33.3 mm to (38.1, 43.2)
- moved HOURS_UNITS 24.7 mm to (45.7, 26.7)
- moved MINUTES_TENS 20.5 mm to (94.0, 8.89)
- moved SECONDS_TENS 14.0 mm to (26.7, 26.7)
- moved SECONDS_UNITS 10.2 mm to (7.62, 26.7)
- moved MINUTES_UNITS 2.54 mm to (64.8, 26.7)
Connections:
- new net HOURS_0: IC5_HOURS_UNITS.3, R48.1
- new net HOURS_1: IC5_HOURS_UNITS.2, R39.1
- new net HOURS_2: IC5_HOURS_UNITS.4, R40.1
- new net HOURS_3: IC5_HOURS_UNITS.7, R41.1
- new net HOURS_4: IC5_HOURS_UNITS.10, R42.1
- new net HOURS_5: D10.C, IC5_HOURS_UNITS.1, R43.1
- new net HOURS_6: IC5_HOURS_UNITS.5, R44.1
- new net HOURS_7: IC5_HOURS_UNITS.6, R45.1
- new net HOURS_8: IC5_HOURS_UNITS.9, R46.1
- new net HOURS_9: IC5_HOURS_UNITS.11, R47.1
- new net INC_HOURS: D8.A, IC4_MINUTES_TENS.5, IC5_HOURS_UNITS.14
- new net INC_HOURS_TENS: IC5_HOURS_UNITS.12, IC6_HOURS_TENS.14
- new net INC_MINUTES: D7.A, IC2_SECONDS_TENS.5, IC3_MINUTES_UNITS.14
- new net INC_MINUTES_TENS: IC3_MINUTES_UNITS.12, IC4_MINUTES_TENS.14
- new net INC_SECONDS_TENS: IC1_SECONDS_UNITS.12, IC2_SECONDS_TENS.14
- new net MASTER_RESET: D1.A, D2.A, D3.A, D4.A, D5.A, D6.A, S1.3
- new net MIN_0: IC3_MINUTES_UNITS.3, R30.1
- new net MIN_1: IC3_MINUTES_UNITS.2, R21.1
- new net MIN_2: IC3_MINUTES_UNITS.4, R22.1
- new net MIN_3: IC3_MINUTES_UNITS.7, R23.1
- new net MIN_4: IC3_MINUTES_UNITS.10, R24.1
- new net MIN_5: IC3_MINUTES_UNITS.1, R25.1
- new net MIN_6: IC3_MINUTES_UNITS.5, R26.1
- new net MIN_7: IC3_MINUTES_UNITS.6, R27.1
- new net MIN_8: IC3_MINUTES_UNITS.9, R28.1
- new net MIN_9: IC3_MINUTES_UNITS.11, R29.1
- new net N$100: D1.C, D8.C, IC4_MINUTES_TENS.15, R56.1
- new net N$102: D4.C, IC3_MINUTES_UNITS.15, R52.1
- new net N$104: D5.C, D9.C, IC6_HOURS_TENS.15, R57.1
- new net N$106: D6.C, IC5_HOURS_UNITS.15, R53.2
- new net N$79: SECONDS_UNITS.7, T7.3
- new net N$80: D2.C, D7.C, IC2_SECONDS_TENS.15, R55.1
- new net N$87: MINUTES_UNITS.7, T22.3
- new net N$88: HOURS_UNITS.7, T38.3
- new net N$89: D3.C, IC1_SECONDS_UNITS.15, R51.1
- new net RESET_HOURS: D10.A, D11.A, D9.A, R58.2
- new net SEC_0: IC1_SECONDS_UNITS.3, R12.1
- new net SEC_1: IC1_SECONDS_UNITS.2, R3.1
- new net SEC_2: IC1_SECONDS_UNITS.4, R4.1
- new net SEC_3: IC1_SECONDS_UNITS.7, R5.1
- new net SEC_4: IC1_SECONDS_UNITS.10, R6.1
- new net SEC_5: IC1_SECONDS_UNITS.1, R7.1
- new net SEC_6: IC1_SECONDS_UNITS.5, R8.1
- new net SEC_7: IC1_SECONDS_UNITS.6, R9.1
- new net SEC_8: IC1_SECONDS_UNITS.9, R10.1
- new net SEC_9: IC1_SECONDS_UNITS.11, R11.1
- new net THOURS_0: IC6_HOURS_TENS.3, R54.1
- new net THOURS_1: IC6_HOURS_TENS.2, R49.1
- new net THOURS_2: D11.C, IC6_HOURS_TENS.4, R50.1
- new net TIME_REFERENCE: CON_TIME_REF.P$1, IC1_SECONDS_UNITS.14
- new net TMIN_0: IC4_MINUTES_TENS.3, R36.1
- new net TMIN_1: IC4_MINUTES_TENS.2, R31.1
- new net TMIN_2: IC4_MINUTES_TENS.4, R32.1
- new net TMIN_3: IC4_MINUTES_TENS.7, R33.1
- new net TMIN_4: IC4_MINUTES_TENS.10, R34.1
- new net TMIN_5: IC4_MINUTES_TENS.1, R35.1
- new net TSEC_0: IC2_SECONDS_TENS.3, R18.1
- new net TSEC_1: IC2_SECONDS_TENS.2, R13.1
- new net TSEC_2: IC2_SECONDS_TENS.4, R14.1
- new net TSEC_3: IC2_SECONDS_TENS.7, R15.1
- new net TSEC_4: IC2_SECONDS_TENS.10, R16.1
- new net TSEC_5: IC2_SECONDS_TENS.1, R17.1
- net GND: now also C1.2, C2.2, C3.2, C4.2, C5.2, C6.2, CON_HIGH_VOLTAGE.P$2, CON_TIME_REF.P$2, IC1_SECONDS_UNITS.13, IC1_SECONDS_UNITS.8, IC2_SECONDS_TENS.13, IC2_SECONDS_TENS.8, IC3_MINUTES_UNITS.13, IC3_MINUTES_UNITS.8, IC4_MINUTES_TENS.13, IC4_MINUTES_TENS.8, IC5_HOURS_UNITS.13, IC5_HOURS_UNITS.8, IC6_HOURS_TENS.13, IC6_HOURS_TENS.8, R51.2, R52.2, R53.1, R55.2, R56.2, R57.2; no longer CON_TUBE_POWER.P$2, HOURS_UNITS.7, MINUTES_UNITS.7, SECONDS_UNITS.7
- net VCC: now also C1.1, C2.1, C3.1, C4.1, C5.1, C6.1, IC1_SECONDS_UNITS.16, IC2_SECONDS_TENS.16, IC3_MINUTES_UNITS.16, IC4_MINUTES_TENS.16, IC5_HOURS_UNITS.16, IC6_HOURS_TENS.16, R58.1, S1.1
- net VHIGH: now also CON_HIGH_VOLTAGE.P$1; no longer CON_TUBE_POWER.P$1
Other:
- board size 182.6 x 80 mm -> 102.5 x 80 mm

Commit message: Start routing for tubes board
Parts:
- moved C6 651.1 mm to (128.3, 83.8), turned to 180 degrees
- moved C5 638.6 mm to (108.0, 83.8), turned to 180 degrees
- moved C4 624.5 mm to (80.0, 83.8), turned to 180 degrees
- moved R58 615.7 mm to (166.4, 68.6)
- moved D11 605.3 mm to (166.4, 64.8)
- moved C3 601.9 mm to (0.00, 83.8), turned to 90 degrees
- moved D9 597.6 mm to (141.0, 80.0), turned to 90 degrees
- moved D10 596.1 mm to (166.4, 61.0)
- moved C2 592.2 mm to (-27.9, 83.8), turned to 90 degrees
- moved C1 583.0 mm to (-74.9, 83.8), turned to 90 degrees
- moved D8 575.5 mm to (94.0, 80.0), turned to 90 degrees
- moved D7 563.6 mm to (-33.0, 100.3), turned to 90 degrees
- moved R57 557.7 mm to (135.9, 81.3), turned to 90 degrees
- moved R55 546.8 mm to (-40.6, 100.3), turned to 90 degrees
- moved R56 542.0 mm to (88.9, 81.3), turned to 90 degrees
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Other:
- board size 102.5 x 80 mm -> 154.6 x 87.6 mm

Commit message: Fix MSPA42 and IN-14 packages
Parts:
- HOURS_TENS, HOURS_UNITS, MINUTES_TENS, MINUTES_UNITS, SECONDS_TENS, SECONDS_UNITS: device russian-nixies:IN-14 -> PGT:IN-14
- moved HOURS_TENS 91.2 mm to (38.1, 11.4), flipped to the top, turned to 0 degrees
- moved T36 64.8 mm to (47.0, 25.4), turned to 90 degrees
- moved HOURS_UNITS 64.5 mm to (43.2, 38.1), flipped to the top
- moved T37 64.2 mm to (40.6, 25.4)
- moved T44 40.0 mm to (99.7, 25.4)
- moved T43 38.7 mm to (99.7, 34.3)
- moved T21 17.8 mm to (7.62, 21.6), turned to 90 degrees
- moved T42 16.5 mm to (101.6, 35.6)
- moved T33 15.9 mm to (99.7, 26.7)
- moved T34 15.9 mm to (99.7, 17.8)
- moved T35 15.9 mm to (99.7, 10.2)
- moved T32 13.3 mm to (99.7, 38.1)
- flipped MINUTES_TENS to the top

Commit message: Group components per digit
Parts:
- moved T6 444.5 mm to (382.3, 47.0), turned to 0 degrees
- moved R8 442.1 mm to (382.3, 58.4)
- moved T7 431.8 mm to (375.9, 47.0), turned to 0 degrees
- moved R3 425.6 mm to (350.5, 58.4)
- moved T1 425.5 mm to (350.5, 47.0), turned to 0 degrees
- moved T8 425.5 mm to (369.6, 47.0), turned to 0 degrees
- moved R9 423.0 mm to (375.9, 58.4)
- moved R10 419.2 mm to (369.6, 58.4)
- moved T2 419.1 mm to (344.2, 47.0), turned to 0 degrees
- moved R11 416.7 mm to (363.2, 58.4)
- moved R4 416.7 mm to (344.2, 58.4)
- moved R1 415.4 mm to (358.1, 34.3)
- moved C1 415.4 mm to (340.4, 73.7)
- moved D3 415.4 mm to (351.8, 90.3)
- moved R51 415.4 mm to (348.0, 90.2)
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Other:
- board size 154.6 x 87.6 mm -> 394 x 128.3 mm

Commit message: Pack layout
Parts:
- moved T6 109.5 mm to (273.1, 39.4)
- moved R8 109.2 mm to (273.1, 55.9)
- moved R9 97.8 mm to (278.1, 55.9)
- moved T7 97.8 mm to (278.1, 44.5)
- moved R1 94.1 mm to (270.5, 68.6), turned to 90 degrees
- moved R3 92.7 mm to (257.8, 55.9)
- moved T1 92.7 mm to (257.8, 44.5)
- moved T2 91.8 mm to (252.7, 39.4)
- moved R4 91.5 mm to (252.7, 55.9)
- moved R5 90.2 mm to (247.7, 55.9)
- moved T3 90.2 mm to (247.7, 44.5)
- moved D3 89.1 mm to (262.9, 96.6)
- moved C1 88.2 mm to (252.7, 83.8)
- moved IC1_SECONDS_UNITS 87.0 mm to (268.0, 83.8)
- moved R51 81.6 mm to (266.7, 97.8)
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Other:
- board size 394 x 128.3 mm -> 305.1 x 128.3 mm

Commit message: Pack more
Parts:
- moved CON_TIME_REF 92.4 mm to (208.3, 116.8)
- moved S1 92.0 mm to (196.8, 123.2)
- moved CON_HIGH_VOLTAGE 85.3 mm to (218.4, 118.1)
- moved R51 81.0 mm to (186.7, 110.5)
- moved R1 79.6 mm to (200.7, 30.5), turned to 0 degrees
- moved T8 78.7 mm to (214.6, 39.4), turned to 315 degrees
- moved T9 77.5 mm to (210.8, 44.5), turned to 315 degrees
- moved R10 77.5 mm to (215.9, 55.9)
- moved R11 76.2 mm to (212.1, 55.9)
- moved T0 76.2 mm to (207.0, 39.4), turned to 315 degrees
- moved SECONDS_UNITS 75.1 mm to (195.6, 19.1)
- moved D3 75.0 mm to (189.2, 110.6)
- moved T7 74.9 mm to (203.2, 44.5), turned to 315 degrees
- moved R12 74.9 mm to (208.3, 55.9)
- moved T6 73.7 mm to (199.4, 39.4), turned to 315 degrees
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Other:
- board size 305.1 x 128.3 mm -> 226.4 x 128.3 mm
